File: pcb_design/testing_pcb/testing_pcb.kicad_pcb (KiCad board)
At the start: 2 copper layers, 60 x 60 mm, 56 parts, among them J1 UART, J10 SOx, J11 Conn_01x04_Pin, J12 Conn_01x04_Pin, J2 ST-LINK Flasher, J3 batt_1x2, J5 INH/Lx, J6 gnd, J7 V, J8 out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

Commit message: fixed error for testing pcb
Parts:
- moved C6 0.51 mm to (161.6, 77.0)
Routing:
- net /VIN_AVDD: track 12.4 -> 54.7 mm, vias 1 -> 3
- net /CP: track 69.4 -> 73.0 mm
- net GND: track 138.4 -> 139.4 mm, vias 25 -> 29
- net /SOA: track 83.7 -> 84.6 mm
- net /SCL: vias 3 -> 4

Commit message: minor changes
Parts:
- renumbered SW2 to BOOT, J1 to GND, SW1 to RESET
Routing:
- net GND: track 139.4 -> 140.9 mm, vias 29 -> 50
- net +3V3: track 196.7 -> 197.6 mm
Other:
- board text added: "+BATT"
- board text added: "-BATT"
- board text added: "3V3"
- board text added: "A"
- board text added: "AVDD"
- board text added: "B"
- board text added: "C"
- board text added: "CP"
- board text added: "CSAREF"
- board text added: "DIR"
- board text added: "FAULT"
- board text added: "GAIN"
- board text added: "GND"
- board text added: "INHA"
- board text added: "INHB"
- board text added: "INHC"
- board text added: "INLA"
- board text added: "INLB"
- board text added: "INLC"
- board text added: "MODE"
- board text added: "O/P"
- board text added: "OUT"
- board text added: "PGO"
- board text added: "RX"
- board text added: "SCL"
- board text added: "SDA"
- board text added: "SLEEP"
- board text added: "SLEW"
- board text added: "SOA"
- board text added: "SOB"
- board text added: "SOC"
- board text added: "SWCLK"
- board text added: "SWDIO"
- board text added: "TX"
- board text added: "VDD_5V"
- board text added: "Vin ADD"
